Commit message: 解决冲突

File: src/openarm_description/urdf/robot/openarm_robot.xacro (robot description, xacro)
@@ -181,18 +181,3 @@
         </xacro:if>
   </xacro:macro>
-<<<<<<< HEAD
-<link name="camera_link">
-    <visual>
-      <geometry><box size="0.02 0.09 0.025"/></geometry>
-      <material name="grey"><color rgba="0.5 0.5 0.5 1"/></material>
-    </visual>
-  </link>
-  <joint name="camera_joint" type="fixed">
-    <parent link="openarm_body_link0"/>
-    <child link="camera_link"/>
-    <origin xyz="0.6 0.0 1.0" rpy="0 0.785 3.1415"/>
-  </joint>
 </robot>
-=======
-</robot>
->>>>>>> aff733e648f7db4132402974620806032e944173
