Commit message: feat: 修改（主要是banana_detector.py，virtual_camera.py以及v10.urdf.xacro中的相机角度）

File: src/openarm_description/urdf/robot/v10.urdf.xacro (robot description, xacro)
@@ -29,46 +29,43 @@
   <xacro:arg name="can_fd" default="true" />
   <xacro:openarm_robot
-  arm_type="v10"
-  body_type="v10"
-  joint_limits="${xacro.load_yaml('$(find openarm_description)/config//arm/v10/joint_limits.yaml')}"
-  inertials="${xacro.load_yaml('$(find openarm_description)/config/arm/v10/inertials.yaml')}"
-  kinematics="${xacro.load_yaml('$(find openarm_description)/config/arm/v10/kinematics.yaml')}"
-  kinematics_link="${xacro.load_yaml('$(find openarm_description)/config/arm/v10/kinematics_link.yaml')}"
-  kinematics_offset="${xacro.load_yaml('$(find openarm_description)/config/arm/v10/kinematics_offset.yaml')}"
-  body_inertials="${xacro.load_yaml('$(find openarm_description)/config/body/v10/inertials.yaml')}"
-  body_kinematics="${xacro.load_yaml('$(find openarm_description)/config/body/v10/kinematics.yaml')}"
-  body_kinematics_link="${xacro.load_yaml('$(find openarm_description)/config/body/v10/kinematics.yaml')}"
-  ee_kinematics_link="${xacro.load_yaml('$(find openarm_description)/config/hand/openarm_hand/kinematics_link.yaml')}"
-  hand="$(arg hand)"
-  ee_type="$(arg ee_type)"
-  ros2_control="$(arg ros2_control)"
-  use_mujoco_hardware="$(arg use_mujoco_hardware)"
-  can_interface="$(arg can_interface)"
-  left_can_interface="$(arg left_can_interface)"
-  right_can_interface="$(arg right_can_interface)"
-  left_arm_prefix="$(arg left_arm_prefix)"
-  right_arm_prefix="$(arg right_arm_prefix)"
-  use_fake_hardware="$(arg use_fake_hardware)"
-  fake_sensor_commands="$(arg fake_sensor_commands)"
-  no_prefix="$(arg no_prefix)"
-  arm_prefix=""
-  body_prefix=""
-  arm_connected_to="base"
-  body_connected_to="world"
-  bimanual="$(arg bimanual)"
-  right_arm_base_xyz="$(arg right_arm_base_xyz)"
-  left_arm_base_xyz="$(arg left_arm_base_xyz)"
-  right_arm_base_rpy="$(arg right_arm_base_rpy)"
-  left_arm_base_rpy="$(arg left_arm_base_rpy)"
-  can_fd="$(arg can_fd)"
+    arm_type="v10"
+    body_type="v10"
+    joint_limits="${xacro.load_yaml('$(find openarm_description)/config//arm/v10/joint_limits.yaml')}"
+    inertials="${xacro.load_yaml('$(find openarm_description)/config/arm/v10/inertials.yaml')}"
+    kinematics="${xacro.load_yaml('$(find openarm_description)/config/arm/v10/kinematics.yaml')}"
+    kinematics_link="${xacro.load_yaml('$(find openarm_description)/config/arm/v10/kinematics_link.yaml')}"
+    kinematics_offset="${xacro.load_yaml('$(find openarm_description)/config/arm/v10/kinematics_offset.yaml')}"
+    body_inertials="${xacro.load_yaml('$(find openarm_description)/config/body/v10/inertials.yaml')}"
+    body_kinematics="${xacro.load_yaml('$(find openarm_description)/config/body/v10/kinematics.yaml')}"
+    body_kinematics_link="${xacro.load_yaml('$(find openarm_description)/config/body/v10/kinematics.yaml')}"
+    ee_kinematics_link="${xacro.load_yaml('$(find openarm_description)/config/hand/openarm_hand/kinematics_link.yaml')}"
+    hand="$(arg hand)"
+    ee_type="$(arg ee_type)"
+    ros2_control="$(arg ros2_control)"
+    use_mujoco_hardware="$(arg use_mujoco_hardware)"
+    can_interface="$(arg can_interface)"
+    left_can_interface="$(arg left_can_interface)"
+    right_can_interface="$(arg right_can_interface)"
+    left_arm_prefix="$(arg left_arm_prefix)"
+    right_arm_prefix="$(arg right_arm_prefix)"
+    use_fake_hardware="$(arg use_fake_hardware)"
+    fake_sensor_commands="$(arg fake_sensor_commands)"
+    no_prefix="$(arg no_prefix)"
+    arm_prefix=""
+    body_prefix=""
+    arm_connected_to="base"
+    body_connected_to="world"
+    bimanual="$(arg bimanual)"
+    right_arm_base_xyz="$(arg right_arm_base_xyz)"
+    left_arm_base_xyz="$(arg left_arm_base_xyz)"
+    right_arm_base_rpy="$(arg right_arm_base_rpy)"
+    left_arm_base_rpy="$(arg left_arm_base_rpy)"
+    can_fd="$(arg can_fd)"
   />
-  <!-- D435 camera mounted on openarm_body_link0 (from MuJoCo openarm_bimanual_cam_v2.xml) -->
   <link name="d435_link">
     <visual>
-      <!-- Approximate pose from MuJoCo: body pos="0.040 0 0.62" -->
-      <origin xyz="0.04 0.0 0.62" rpy="3.14 0.78 1.57"/>
+      <origin xyz="0.04 0.0 0.62" rpy="3.14 1.3 0"/>
       <geometry>
-        <!-- Use D435 mesh from openarm_mujoco (under v1/meshes/visual/cam) -->
-        <mesh filename="file:///home/zjc/openarm_ws/openarm_mujoco/v1/meshes/visual/cam/d435_0.stl"/>
+        <mesh filename="file:///home/ros/openarm_ws/openarm_mujoco/v1/meshes/visual/cam/d435_0.stl"/>
       </geometry>
       <material name="d435_material">
@@ -77,5 +74,5 @@
     </visual>
     <collision>
-      <origin xyz="0.04 0.0 0.62" rpy="3.14 0.78 1.57"/>
+      <origin xyz="0.04 0.0 0.62" rpy="3.14 1.3 0"/>
       <geometry>
         <box size="0.05 0.05 0.05"/>
@@ -86,21 +83,16 @@
     <parent link="openarm_body_link0"/>
     <child link="d435_link"/>
-    <origin xyz="0.04 0.0 0.62" rpy="3.14 0.78 1.57"/>
+    <origin xyz="0.04 0.0 0.62" rpy="3.14 1.3 0"/>
   </joint>
-  <!-- Optical frame for D435 (standard ROS camera frame: x right, y down, z forward) -->
   <link name="d435_optical_frame"/>
   <joint name="d435_optical_joint" type="fixed">
     <parent link="d435_link"/>
     <child link="d435_optical_frame"/>
-    <!-- rotation: Rz(-90deg) * Rx(-90deg) -->
     <origin xyz="0 0 0" rpy="-1.5707963 0 -1.5707963"/>
   </joint>
-  <!-- Static table under world for visualization in RViz -->
   <link name="table">
     <visual>
-      <!-- Match MuJoCo table position: pos="0.35 0 0.15" -->
       <origin xyz="0.35 0 0.15" rpy="0 0 0"/>
       <geometry>
-        <!-- Size corresponds to MuJoCo half-sizes: 0.25 0.3 0.15 -->
         <box size="0.5 0.6 0.3"/>
       </geometry>
@@ -120,14 +112,17 @@
     <child link="table"/>
   </joint>
-  <!-- Static banana mesh on table for visualization in RViz -->
   <link name="banana">
     <visual>
-      <!-- Match MuJoCo banana pose: pos="0.35 0 0.35" euler="0 0 1.57" -->
       <origin xyz="0.35 0 0.35" rpy="0 0 1.57"/>
       <geometry>
-        <!-- Absolute path to banana mesh in openarm_mujoco -->
-        <mesh filename="file:///home/zjc/openarm_ws/openarm_mujoco/v1/meshes/011_banana/textured_simple.obj"/>
+        <mesh filename="file:///home/ros/openarm_ws/openarm_mujoco/v1/meshes/011_banana/textured_simple.obj"/>
       </geometry>
     </visual>
+    <collision>
+      <origin xyz="0.35 0 0.35" rpy="0 0 1.57"/>
+      <geometry>
+        <box size="0.04 0.04 0.15"/>
+      </geometry>
+    </collision>
   </link>
   <joint name="world_to_banana" type="fixed">

Commit message: 路径修改

File: src/openarm_description/urdf/robot/v10.urdf.xacro (robot description, xacro)
@@ -116,5 +116,5 @@
       <origin xyz="0.35 0 0.35" rpy="0 0 1.57"/>
       <geometry>
-        <mesh filename="file:///home/zcj/openarm_ws/openarm_mujoco/v1/meshes/011_banana/textured_simple.obj"/>
+        <mesh filename="file:///home/zjc/openarm_ws/openarm_mujoco/v1/meshes/011_banana/textured_simple.obj"/>
       </geometry>
     </visual>

Commit message: Fix: 修复相机物理位置，同步虚拟相机脚本，去除算法人工补丁

File: src/openarm_description/urdf/robot/v10.urdf.xacro (robot description, xacro)
@@ -65,5 +65,5 @@
   <link name="d435_link">
     <visual>
-      <origin xyz="0.04 0.0 0.62" rpy="3.14 1.3 0"/>
+      <origin xyz="0 0 0" rpy="1.57 0 1.57"/>
       <geometry>
         <mesh filename="file:///home/ros/openarm_ws/openarm_mujoco/v1/meshes/visual/cam/d435_0.stl"/>
@@ -74,5 +74,5 @@
     </visual>
     <collision>
-      <origin xyz="0.04 0.0 0.62" rpy="3.14 1.3 0"/>
+      <origin xyz="0 0 0" rpy="0 0 0"/>
       <geometry>
         <box size="0.05 0.05 0.05"/>
@@ -83,5 +83,5 @@
     <parent link="openarm_body_link0"/>
     <child link="d435_link"/>
-    <origin xyz="0.04 0.0 0.62" rpy="3.14 1.3 0"/>
+    <origin xyz="0.2 0 0.8" rpy="3.14 1.57 0"/>
   </joint>
   <link name="d435_optical_frame"/>
@@ -114,5 +114,5 @@
   <link name="banana">
     <visual>
-      <origin xyz="0.35 0 0.35" rpy="0 0 1.57"/>
+      <origin xyz="0 0 0" rpy="0 0 1.57"/>
       <geometry>
         <mesh filename="file:///home/ros/openarm_ws/openarm_mujoco/v1/meshes/011_banana/textured_simple.obj"/>
@@ -120,5 +120,5 @@
     </visual>
     <collision>
-      <origin xyz="0.35 0 0.35" rpy="0 0 1.57"/>
+      <origin xyz="0 0 0" rpy="0 0 1.57"/>
       <geometry>
         <box size="0.04 0.04 0.15"/>
@@ -129,4 +129,5 @@
     <parent link="world"/>
     <child link="banana"/>
+    <origin xyz="0.35 0 0.35" rpy="0 0 0"/>
   </joint>
 </robot>
